File: bbbalarm.kicad_sch (KiCad schematic)
At the start: 34 parts, among them J101 IN0, J102 PWR, J103 IN1, J104 PIR0, J105 PIR1, P8 BeagleBone_Black_Header, P9 BeagleBone_Black_Header, SW101 Reset, SW102 PWR, U101 HCPL-263N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

Commit message: Add Temp sensor and serial header
Signed-off-by: Benedikt Spranger <b.spranger@linutronix.de>
Parts:
- added J106: serial, Connector_PinHeader_2.54mm:PinHeader_1x03_P2.54mm_Vertical, symbol Connector_Generic:Conn_01x03
- added R113: 1k, Resistor_SMD:R_0402_1005Metric, symbol Device:R
- added U102: SHT35-DIS, Sensor_Humidity:Sensirion_DFN-8-1EP_2.5x2.5mm_P0.5mm_EP1.1x1.7mm, symbol Sensor_Humidity:SHT35-DIS
- D114, J101, J102, J103, J104, J105, R109, R110, R111, R112, U101, U104: assemble (none) -> n
- P8, P9, SW101, SW102: assemble y -> n
- R105, R106, R107, R108: LCSC C11702 -> (none); ManuPart# 0402WGF1001TCE -> (none); Manufacture UNI-ROYAL(Uniroyal Elec) -> (none); assemble y -> n
Connections:
- net +3V3: now also U102.5 (VDD)
- net GNDD: now also J106.1 (Pin_1), U102.2 (ADDR), U102.7 (R), U102.8 (VSS), U102.9 (VSS)
- net SCL: now also U102.4 (SCL)
- net SDA: now also U102.1 (SDA)
- net RX: now reaches P9.11 (Pin_11)
- net RX: now also J106.2 (Pin_2)
- net TX: now reaches P9.13 (Pin_13)
- net TX: now also J106.3 (Pin_3)
- net ALERT: now reaches P8.15 (Pin_15)
- net ALERT: now also U102.3 (ALERT)
- net nRST: now reaches P8.17 (Pin_17)
- net nRST: now also R113.1
- new net: R113.2, U102.6 (~{RESET})
- no-connect marks 64 -> 60
Other:
- moved on the sheet: D101, D102, D103, D104, R105, R106, R107, R108

Commit message: Revisit Parts
Parts:
- C101: DistribPart# (none) -> C1525; Distributor (none) -> JLPCB; LCSC C1525 -> (none); LCSC# (none) -> C1525
- D101, D102: value LED -> LED red; DistribPart# (none) -> OSR5JA34E4A; Distributor (none) -> TME; LCSC C2286 -> (none); LCSC# (none) -> C2286; ManuPart# KT-0603R -> OSR5JA34E4A; Manufacture Hubei KENTO Elec -> OPTOSUPPLY; assemble y -> n
- D103, D104: value LED -> LED green; DistribPart# (none) -> OSG5TA34E4A; Distributor (none) -> TME; LCSC C2286 -> (none); LCSC# (none) -> C2286; ManuPart# KT-0603R -> OSG5TA34E4A; Manufacture Hubei KENTO Elec -> OPTOSUPPLY; assemble y -> n
- D114: DistribPart# (none) -> 1N4004-DIO; Distributor (none) -> TME; ManuPart# (none) -> 1N4004; Manufacture (none) -> DIOTEC SEMICONDUCTOR
- J101, J102, J103, J104, J105, J106, P8, P9, R105, R106, R107, R108, R109, R110, R111, R112, SW101, SW102, U101: Distributor (none) -> TME
- JP105, JP106, JP107, JP108: Distributor (none) -> N/A
- R101, R102, R103, R104, R113: DistribPart# (none) -> C11702; Distributor (none) -> JLPCB; LCSC C11702 -> (none); LCSC# (none) -> C11702
- U102: DistribPart# (none) -> C90161; Distributor (none) -> JLPCB; LCSC C90161 -> (none); LCSC# (none) -> C90161
- U103: DistribPart# (none) -> C6482; Distributor (none) -> JLPCB; LCSC C6482 -> (none); LCSC# (none) -> C6482
- U104: DistribPart# (none) -> TSN1-2450; Distributor (none) -> TME; ManuPart# (none) -> TSN 1-2450
